File: zak180/vga.kicad_sch (KiCad schematic)
At the start: 31 parts, among them J3 DE15_Receptacle_HighDensity_M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, Q1 BC547, U10 6264, U12 74HC574, U13 74HC174, U14 2764, U15 74HC166, U4 74HC244, U5 XC9536PC44, U6 74HC244, U7 74HC02, U8 74HC04, U9 74HC245

Commit message: HW: Further work on schematic
Parts:
- removed U8: 74HC04, Package_DIP:DIP-14_W7.62mm, symbol 74xx:74HC04
Connections:
- net GND: no longer U7.5, U7.6
- net at U10.22 (~{OE}), U7.1: now also U7.5, U7.6
- net at U7.4: now also U10.27 (~{WR})
- net ~{VBLANK} renamed VBLANK
- no-connect marks 19 -> 18
Other:
- moved on the sheet: U7B

Commit message: HW: Change RAM to static
Parts:
- U6: footprint (none) -> Package_DIP:DIP-20_W7.62mm
Changed lines of the file:
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@@
 			)
 		)
-		(property "Footprint" ""
+		(property "Footprint" "Package_DIP:DIP-20_W7.62mm"
 			(at 87.63 156.21 0)
 			(effects
