File: zak180/floppy.kicad_sch (KiCad schematic)
At the start: 15 parts, among them J1 Conn_02x17_Odd_Even, J6 Floppy Power, U1 82077AA/PC8477, Y1 24 MHz

Commit message: HW: PCB complete
Connections:
- net GND: no longer U1.27 (IDENT)
- net VCC: now also U1.27 (IDENT)
Changed lines of the file:
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@@
 	)
 	(junction
+		(at 105.41 127)
+		(diameter 0)
+		(color 0 0 0 0)
+	)
+	(junction
 		(at 219.71 96.52)
 		(diameter 0)
@@
 	)
 	(junction
-		(at 105.41 134.62)
-		(diameter 0)
-		(color 0 0 0 0)
-	)
-	(junction
 		(at 129.54 151.13)
 		(diameter 0)
@@
 	(wire
 		(pts
-			(xy 102.87 125.73) (xy 102.87 132.08)
+			(xy 105.41 125.73) (xy 105.41 127)
 		)
 		(stroke
@@
 	(wire
 		(pts
-			(xy 106.68 132.08) (xy 102.87 132.08)
+			(xy 106.68 132.08) (xy 105.41 132.08)
 		)
 		(stroke
@@
 	(wire
 		(pts
-			(xy 105.41 134.62) (xy 105.41 127)
-		)
-		(stroke
-			(width 0)
-			(type default)
-		)
-	)
-	(wire
-		(pts
 			(xy 219.71 99.06) (xy 219.71 104.14)
 		)
@@
 	(wire
 		(pts
+			(xy 105.41 127) (xy 105.41 132.08)
+		)
+		(stroke
+			(width 0)
+			(type default)
+		)
+	)
+	(wire
+		(pts
 			(xy 147.32 121.92) (xy 168.91 121.92)
 		)
@@
 	(wire
 		(pts
-			(xy 105.41 127) (xy 106.68 127)
-		)
-		(stroke
-			(width 0)
-			(type default)
-		)
-	)
-	(wire
-		(pts
 			(xy 171.45 63.5) (xy 147.32 63.5)
 		)
@@
 	(wire
 		(pts
+			(xy 105.41 127) (xy 106.68 127)
+		)
+		(stroke
+			(width 0)
+			(type default)
+		)
+	)
+	(wire
+		(pts
 			(xy 219.71 73.66) (xy 219.71 76.2)
 		)
@@
 	(symbol
 		(lib_id "power:VCC")
-		(at 102.87 125.73 0)
+		(at 105.41 125.73 0)
 		(unit 1)
 		(exclude_from_sim no)
@@
 		(dnp no)
 		(property "Reference" "#PWR09"
-			(at 102.87 129.54 0)
+			(at 105.41 129.54 0)
 			(effects
 				(font
@@
 		)
 		(property "Value" "VCC"
-			(at 99.568 125.73 0)
+			(at 102.108 125.73 0)
 			(effects
 				(font
@@
 		)
 		(property "Footprint" ""
-			(at 102.87 125.73 0)
+			(at 105.41 125.73 0)
 			(effects
 				(font
@@
 		)
 		(property "Datasheet" ""
-			(at 102.87 125.73 0)
+			(at 105.41 125.73 0)
 			(effects
 				(font
@@
 		)
 		(property "Description" "Power symbol creates a global label with name \"VCC\""
-			(at 102.87 125.73 0)
+			(at 105.41 125.73 0)
 			(effects
 				(font
