File: zak180/memory.kicad_sch (KiCad schematic)
At the start: 28 parts, among them U28 TC511000AP, U29 TC511000AP, U30 TC511000AP, U31 TC511000AP, U32 TC511000AP, U33 TC511000AP, U34 TC511000AP, U35 TC511000AP, U36 74HC157, U37 74HC157, U38 74HC157, U39 74HC04

Commit message: HW: Before abandoning DRAM
Parts:
- removed unit 6 of U39
- removed unit 5 of U39
- added C70, C71: 47p, Capacitor_THT:C_Disc_D4.3mm_W1.9mm_P5.00mm, symbol Device:C
- added R40, R41: 330R, Resistor_THT:R_Axial_DIN0207_L6.3mm_D2.5mm_P7.62mm_Horizontal, symbol Device:R
- added U40: AS6C4008-55PCN, Package_DIP:DIP-32_W15.24mm, symbol Memory_RAM:AS6C4008-55PCN
- added U41: 74HC04, symbol 74xx:74HC04
Connections:
- net GND: now also C70.1, C71.1
- new net: R40.1, U41.2
- new net: C70.2, R40.2, U41.3
- new net: R41.1, U41.6
- new net: C71.2, R41.2, U41.9
- new net ~{REFSH}: U41.1
- no-connect marks 4 -> 2
Other:
- moved on the sheet: C58, C59, C60, C61, C62, C63, C64, C65, C66, C67, C68, C69

Commit message: HW: Change RAM to static
Parts:
- removed R38, R39, R40, R41: 330R, Resistor_THT:R_Axial_DIN0207_L6.3mm_D2.5mm_P7.62mm_Horizontal, symbol Device:R
- removed U28, U29, U30, U31, U32, U33, U34, U35: TC511000AP, Package_DIP:DIP-18_W7.62mm, symbol 8bits:TC511000AP
- removed U36, U37, U38: 74HC157, Package_DIP:DIP-16_W7.62mm, symbol 74xx:74LS157
- removed U39, U41: 74HC04, symbol 74xx:74HC04
- added U28: AS6C4008-55PCN, Package_DIP:DIP-32_W15.24mm, symbol Memory_RAM:AS6C4008-55PCN
- added U29: 27C128, Package_DIP:DIP-28_W15.24mm, symbol Memory_EPROM:27C128
- added U30: 74HC00, Package_DIP:DIP-14_W7.62mm, symbol 74xx:74HC00
- C56, C57, C70, C71: value 47p -> 100n; footprint Capacitor_THT:C_Disc_D4.3mm_W1.9mm_P5.00mm -> Capacitor_THT:C_Disc_D5.0mm_W2.5mm_P2.50mm
Connections:
- net A0: now also U40.12 (A0), U28.12 (A0), U29.10 (A0)
- net A1: now also U40.11 (A1), U28.11 (A1), U29.9 (A1)
- net A10: now also U40.23 (A10), U28.23 (A10), U29.21 (A10)
- net A11: now also U40.25 (A11), U28.25 (A11), U29.23 (A11)
- net A12: now also U40.4 (A12), U28.4 (A12), U29.2 (A12)
- net A13: now also U40.28 (A13), U28.28 (A13), U29.26 (A13)
- net A14: now also U40.3 (A14), U28.3 (A14)
- net A15: now also U40.31 (A15), U28.31 (A15)
- net A16: now also U40.2 (A16), U28.2 (A16)
- net A17: now also U40.30 (A17), U28.30 (A17)
- net A18: now also U40.1 (A18), U28.1 (A18)
- net A19: now also U30.1, U30.10, U30.2
- net A2: now also U40.10 (A2), U28.10 (A2), U29.8 (A2)
- net A3: now also U40.9 (A3), U28.9 (A3), U29.7 (A3)
- net A4: now also U40.8 (A4), U28.8 (A4), U29.6 (A4)
- net A5: now also U40.7 (A5), U28.7 (A5), U29.5 (A5)
- net A6: now also U40.6 (A6), U28.6 (A6), U29.4 (A6)
- net A7: now also U40.5 (A7), U28.5 (A7), U29.3 (A7)
- net A8: now also U40.27 (A8), U28.27 (A8), U29.25 (A8)
- net A9: now also U40.26 (A9), U28.26 (A9), U29.24 (A9)
- net D0: now also U40.13 (DQ0), U28.13 (DQ0), U29.11 (D0)
- net D1: now also U40.14 (DQ1), U28.14 (DQ1), U29.12 (D1)
- net D2: now also U40.15 (DQ2), U28.15 (DQ2), U29.13 (D2)
- net D3: now also U40.17 (DQ3), U28.17 (DQ3), U29.15 (D3)
- net D4: now also U40.18 (DQ4), U28.18 (DQ4), U29.16 (D4)
- net D5: now also U40.19 (DQ5), U28.19 (DQ5), U29.17 (D5)
- net D6: now also U40.20 (DQ6), U28.20 (DQ6), U29.18 (D6)
- net D7: now also U40.21 (DQ7), U28.21 (DQ7), U29.19 (D7)
- net GND: now also C56.2, C57.2, C70.2, C71.2, U40.16 (VSS), U28.16 (VSS), U29.14 (GND), U30.7 (GND); no longer C56.1, C57.1, C70.1, C71.1
- net VCC: now also C56.1, C57.1, C70.1, C71.1, U40.32 (VCC), U28.32 (VCC), U29.1 (VPP), U29.27 (~{PGM}), U29.28 (VCC), U30.14 (VCC)
- net ~{WR}: now also U40.29 (WE#), U28.29 (WE#)
- net at U40.22 (CE#): now also U30.6
- net ~{RD}: now reaches U40.24 (OE#)
- net ~{RD}: now also U28.24 (OE#), U29.22 (~{OE})
- new net: U28.22 (CE#), U30.8
- new net: U30.3, U30.4
- new net: U30.11, U30.5, U30.9
- new net ~{RAM}: U30.12, U30.13
- new net ~{ROM}: U29.20 (~{CE})
- no-connect marks 2 -> 0
Other:
- moved on the sheet: U40

Commit message: HW: PCB complete
Parts:
- removed C58, C59, C60, C61, C62, C63, C64, C65, C66, C67, C68, C69: 100n, Capacitor_THT:C_Disc_D5.0mm_W2.5mm_P2.50mm, symbol Device:C
