File: zak180/zak180.kicad_sch (KiCad schematic)
At the start: 5 parts, among them U16 74HC00

Commit message: HW: PCB complete
Parts:
- added H1, H2, H3, H4: MountingHole_Pad, MountingHole:MountingHole_3.2mm_M3_Pad_Via, symbol Mechanical:MountingHole_Pad
Connections:
- net GND: now also H1.1, H2.1, H3.1, H4.1
