File: kicad/serial.kicad_sch (KiCad schematic)
At the start: 14 parts, among them J7 DE9_Plug_MountingHoles, J8 USB_C_Receptacle_USB2.0_14P, U25 MAX232, U26 CH340N

Commit message: hw: simplify logic, replace some SSI with GALs
Changed lines of the file:
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@@
 (kicad_sch
-	(version 20231120)
+	(version 20250114)
 	(generator "eeschema")
-	(generator_version "8.0")
+	(generator_version "9.0")
 	(paper "A4")
 	(junction
@@
 		(shape input)
 		(at 119.38 138.43 0)
-		(fields_autoplaced yes)
 		(effects
 			(font
@@
 		(shape output)
 		(at 119.38 135.89 0)
-		(fields_autoplaced yes)
 		(effects
 			(font
@@
 		(shape input)
 		(at 93.98 71.12 180)
-		(fields_autoplaced yes)
 		(effects
 			(font
@@
 		(shape output)
 		(at 93.98 81.28 180)
-		(fields_autoplaced yes)
 		(effects
 			(font
@@
 		(shape input)
 		(at 93.98 76.2 180)
-		(fields_autoplaced yes)
 		(effects
 			(font
@@
 		(shape output)
 		(at 93.98 86.36 180)
-		(fields_autoplaced yes)
 		(effects
 			(font
