File: kicad/serial.kicad_sch (KiCad schematic)
At the start: 14 parts, among them J7 DE9_Plug_MountingHoles, J8 USB_C_Receptacle_USB2.0_14P, U25 MAX232, U26 CH340N

Commit message: hw: finish schematic, start routing
Parts:
- J7: value DE9_Plug_MountingHoles -> DSUB-9; footprint Connector_Dsub:DSUB-9_Male_Horizontal_P2.77x2.84mm_EdgePinOffset7.70mm_Housed_MountingHolesOffset9.12mm -> Connector_Dsub:DSUB-9_Socket_Horizontal_P2.77x2.84mm_EdgePinOffset4.94mm_Housed_MountingHolesOffset4.94mm
- J8: value USB_C_Receptacle_USB2.0_14P -> USB C
Other:
- company: (none) -> A.K.
- title: (none) -> UART
- moved on the sheet: C52, C53, C54, C55, J8, R34, R35, U26
