File: kicad/sound.kicad_sch (KiCad schematic)
At the start: 18 parts, among them J4 Speaker, U11 74HC02, U16 74HC00, U17 LM386, U27 74HC32, U3 PSG_AY-3-8912

Commit message: hw: simplify logic, replace some SSI with GALs
Parts:
- removed U27: 74HC32, Package_DIP:DIP-14_W7.62mm, symbol 74xx:74LS32
- added unit 5 of U16
- added unit 3 of U16
Connections:
- net A0: now also U11.9
- net GND: now also U16.7 (GND); no longer U11.8, U11.9
- net VCC: now also U16.14 (VCC)
- net ~{CS}: now also U11.8
- net at U11.11: now also U16.8
- net at U11.10: now also U16.10, U16.9
- no-connect marks 5 -> 4
Other:
- moved on the sheet: U11C
