File: kicad/floppy.kicad_sch (KiCad schematic)
At the start: 15 parts, among them J1 Conn_02x17_Odd_Even, J6 Floppy Power, U1 82077AA/PC8477, Y1 24 MHz

Commit message: hw: finish schematic, start routing
Other:
- company: (none) -> A.K.
Changed lines of the file:
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@@
 	(generator_version "9.0")
 	(paper "A4")
+	(title_block
+		(date "2025-06-18")
+		(rev "A")
+		(company "A.K.")
+	)
 	(rectangle
 		(start 210.82 121.92)
