File: kicad/cf.kicad_sch (KiCad schematic)
At the start: 4 parts

Commit message: hw: finish routing
Parts:
- J3: value ~ -> Compact Flash
- R19: value 560R -> 1K
Changed lines of the file:
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@@
 			)
 		)
-		(property "Value" "~"
-			(at 140.97 52.07 0)
+		(property "Value" "Compact Flash"
+			(at 150.622 52.578 0)
 			(effects
 				(font
@@
 			)
 		)
-		(property "Value" "560R"
+		(property "Value" "1K"
 			(at 168.91 96.5199 0)
 			(effects
