File: kicad/clock.kicad_sch (KiCad schematic)
At the start: 16 parts, among them J9 Reset, Q2 BC547, SW1 Reset, U18 NE555P, U19 74HC163, X1 25.175 MHz

Commit message: hw: finish schematic, start routing
Parts:
- removed C37: 100n, Capacitor_THT:C_Disc_D5.0mm_W2.5mm_P2.50mm, symbol Device:C
- removed U19: 74HC163, Package_DIP:DIP-16_W7.62mm, symbol 74xx:74LS163
Connections:
- net RST: no longer names the net of R32.1, U18.3 (Q)
- no-connect marks 4 -> 0
Other:
- company: (none) -> A.K.
- title: (none) -> Clock and reset
- moved on the sheet: C35, C36, X1
