File: kicad/keyboard.kicad_sch (KiCad schematic)
At the start: 3 parts, among them J5 Conn_02x06_Odd_Even, U22 74HC244

Commit message: hw: finish schematic, start routing
Other:
- company: (none) -> A.K.
- title: (none) -> Keyboard
Changed lines of the file:
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@@
 	(generator_version "9.0")
 	(paper "A4")
+	(title_block
+		(title "Keyboard")
+		(date "2025-06-18")
+		(rev "A")
+		(company "A.K.")
+	)
 	(text "Designed to work with:\nhttps://github.com/agkaminski/keyboard2"
 		(exclude_from_sim no)

Commit message: hw: finish routing
Parts:
- J5: value Conn_02x06_Odd_Even -> Keyboard
Changed lines of the file:
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@@
 			)
 		)
-		(property "Value" "Conn_02x06_Odd_Even"
+		(property "Value" "Keyboard"
 			(at 134.62 83.82 0)
 			(effects
