File: kicad/pio.kicad_sch (KiCad schematic)
At the start: 5 parts, among them J2 DB25_Receptacle_MountingHoles, U2 Z80 PIO A

Commit message: Fix wrong D-SUB footprints, rev C
Parts:
- J2: footprint Connector_Dsub:DSUB-25_Pins_Horizontal_P2.77x2.84mm_EdgePinOffset4.94mm_Housed_MountingHolesOffset4.94mm -> Connector_Dsub:DSUB-25_Socket_Horizontal_P2.77x2.84mm_EdgePinOffset9.90mm_Housed_MountingHolesOffset11.32mm
Changed lines of the file:
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@@
 	(title_block
 		(title "User port")
-		(date "2025-07-03")
-		(rev "B")
+		(date "2025-07-20")
+		(rev "C")
 		(company "A.K.")
 	)
@@
 			)
 		)
-		(property "Footprint" "Connector_Dsub:DSUB-25_Pins_Horizontal_P2.77x2.84mm_EdgePinOffset4.94mm_Housed_MountingHolesOffset4.94mm"
+		(property "Footprint" "Connector_Dsub:DSUB-25_Socket_Horizontal_P2.77x2.84mm_EdgePinOffset9.90mm_Housed_MountingHolesOffset11.32mm"
 			(at 198.12 96.52 0)
 			(effects

Commit message: rev D
- Fix SUB-D footprints yet again,
- rotate keyboard connector to remove cable twist,
- add onboard speaker.
Parts:
- J2: footprint Connector_Dsub:DSUB-25_Socket_Horizontal_P2.77x2.84mm_EdgePinOffset9.90mm_Housed_MountingHolesOffset11.32mm -> Connector_Dsub:DSUB-25_Socket_Horizontal_P2.77x2.84mm_EdgePinOffset7.70mm_Housed_MountingHolesOffset9.12mm
Changed lines of the file:
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@@
 	(title_block
 		(title "User port")
-		(date "2025-07-20")
-		(rev "C")
+		(date "2025-08-02")
+		(rev "D")
 		(company "A.K.")
 	)
@@
 			)
 		)
-		(property "Footprint" "Connector_Dsub:DSUB-25_Socket_Horizontal_P2.77x2.84mm_EdgePinOffset9.90mm_Housed_MountingHolesOffset11.32mm"
+		(property "Footprint" "Connector_Dsub:DSUB-25_Socket_Horizontal_P2.77x2.84mm_EdgePinOffset7.70mm_Housed_MountingHolesOffset9.12mm"
 			(at 198.12 96.52 0)
 			(effects
