File: kicad/zak181.kicad_sch (KiCad schematic)
At the start: 10 parts, among them U11 74HC02, U16 74HC00

Commit message: hw: finish schematic, start routing
Parts:
- removed U11: 74HC02, Package_DIP:DIP-14_W7.62mm, symbol 74xx:74HC02
- removed U16: 74HC00, Package_DIP:DIP-14_W7.62mm, symbol 74xx:74HC00
Connections:
- no-connect marks 5 -> 3
Other:
- removed sheet floppy
- added sheet cf (cf.kicad_sch)
- sheet clock ports: added none; removed 1.57 MHz, RST
- sheet cpu ports: added ~{CF}; removed ~{FLOPPY}
- sheet sound ports: added A, SCROLL[5..0], ~{A}; removed none
- sheet vga ports: added A[13..0], SCROLL[5..0], ~{IRQACK}, ~{IRQ}; removed A[12..0], VBLANK
- company: (none) -> A.K.
- title: (none) -> ZAK181 Single Board Computer
